File: EPICS elephant project/EPICS elephant project.kicad_sch (KiCad schematic)
At the start: 29 parts, among them U1 LM358AD, U2 LM358AD, U3 LM324N, U4 AD620ANZ, U5 LM324N, U6 ESP32-DevKitC

Commit message: tried to figure out how to simulate it
didnt work lots of errors
Parts:
- added V1: VSIN, symbol Simulation_SPICE:VSIN
- added V2: 5, symbol Simulation_SPICE:VDC
- added V3: -5, symbol Simulation_SPICE:VDC
- R5: value R_Variable -> 10k
Connections:
- net GND: no longer C2.2, R4.2, R7.1, U2.4 (GND), U3.11 (GND), U5.11 (GND)
- net VCC +5v: now also V2.1
- net VEE -5v: now also R4.2, U2.4 (GND), U3.11 (GND), U5.11 (GND), V3.1
- net +Vin: no longer names the net of R10.1
- net +Vin: now also V1.2
- net -Vin: no longer names the net of R11.1
- net -Vin: now also V1.1
- new net 0: C2.2, R7.1, V2.2, V3.2
