File: EPICS elephant project/EPICS elephant project.kicad_pcb (KiCad board)
At the start: 2 copper layers, 100 x 54.6 mm, 33 parts, among them U1 LM358AD, U2 LM358AD, U3 LM324N, U4 AD620ANZ, U5 LM324N, U6 ESP32-DevKitC

Commit message: Added Updated_Schematic
The working directory for now. Will update / change when needed
Parts:
- added G***: LOGO, LOGO, F.Cu at (152.6, 97.8)
- moved R10 0.34 mm to (189.2, 78.1)
- moved R9 0.34 mm to (185.3, 85.7)
Other:
- board text added: "EPICS Elephant Project"
