File: circuitSPICEsimulation/circuitSPICEsimulation.kicad_sch (KiCad schematic)
At the start: 31 parts, among them U1 ${SIM.PARAMS}, U2 ${SIM.PARAMS}, U3 ${SIM.PARAMS}, U4 ${SIM.PARAMS}, U6 ${SIM.PARAMS}

Commit message: Added Updated_Schematic
The working directory for now. Will update / change when needed
Parts:
- C3: value 100nF -> 70nF
Connections:
- net at C1.2, R8.2, U2.5: no longer R13.1
Changed lines of the file:
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@@
-	(wire
-		(pts
-			(xy 219.71 49.53) (xy 231.14 49.53)
-		)
-		(stroke
-			(width 0)
-			(type default)
-		)
-	)
 	(wire
 		(pts
@@
 			)
 		)
-		(property "Value" "100nF"
+		(property "Value" "70nF"
 			(at 320.04 82.55 90)
 			(effects
